File: kimchi_usb_ulid.kicad_pcb (KiCad board)
At the start: 4 copper layers, 65 x 32 mm, 44 parts, among them J1 DF40HC(3.5)-60DS, J2 DF40HC(3.5)-60DS, J3 USB_A, J4 USB_A, J5 USB_A, U1 24C32, U2 AP2152A, U3 AP2152A, U4 USB2514B_Bi, Y1 24MHz 50 PPM

Commit message: Change mask web to 3 mil
Other:
- rule solder_mask_min_width: 0.1016 -> 0.0762
Changed lines of the file:
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@@
     (pad_drill 0)
     (pad_to_mask_clearance 0.0508)
-    (solder_mask_min_width 0.1016)
+    (solder_mask_min_width 0.0762)
     (aux_axis_origin 107 126)
     (grid_origin 107 126)
