File: kimchi_usb_ulid.sch (KiCad schematic (older format))
At the start: 44 parts, among them J1 DF40HC(3.5)-60DS, J2 DF40HC(3.5)-60DS, J3 USB_A, J4 USB_A, J5 USB_A, U1 24C32, U2 AP2152A, U3 AP2152A, U4 USB2514B_Bi, Y1 24MHz 50 PPM

Commit message: Finish bom
Parts:
- C1, C2: Mfgr (none) -> Murata; Mfgrpart (none) -> GCM1555C1H180FA16D; Vendorpart (none) -> 490-16457-1-ND
- C10: Mfgrpart (none) -> GRM155R60J475ME87D; Part GRM155R60J475ME87D -> (none)
- C11, C12, C13, C4, C5, C6, C7, C8, C9: Mfgrpart (none) -> GRM155R71E104ME14D; Part GRM155R71E104ME14D -> (none)
- C3: Mfgrpart (none) -> GRM155C81A105KA12D; Part GRM155C81A105KA12D -> (none)
- D1, D2, D3: Mfgrpart (none) -> SZESD7205DT5G; Part SZESD7205DT5G -> (none)
- H1, H2, H3, H4, LOGO1: Populate (none) -> DNP
- J1, J2: Mfgr (none) -> Hirose; Mfgrpart (none) -> DF40HC(3.5)-60DS-0.4V(51); Vendorpart (none) -> H11917CT-ND
- J3, J4, J5: Mfgr (none) -> Stewart; Mfgrpart (none) -> SS-52100-001; Vendorpart (none) -> 380-1412-ND
- R1: Mfgr (none) -> Yageo; Mfgrpart (none) -> RC0402JR-0710KL; Vendorpart (none) -> 311-10KJRCT-ND
- R10, R11, R12, R13, R2, R3, R6, R8, R9: Mfgrpart (none) -> RC0402FR-07100KL; Part RC0402FR-07100KL -> (none)
- R4: Mfgrpart (none) -> RC0402FR-0712KL; Part RC0402FR-0712KL -> (none)
- R5, R7: Mfgrpart (none) -> RC0402JR-070RL; Part RC0402JR-070RL -> (none)
- U1: Mfgrpart (none) -> M24C32-FMC6TG; Part M24C32-FMC6TG -> (none)
- U2, U3: Mfgr (none) -> Diodes; Mfgrpart (none) -> AP2152AFGEG-7; Vendorpart (none) -> AP2152AFGEG-7DICT-ND
- U4: Mfgr (none) -> Microchip; Mfgrpart (none) -> USB2514B-AEZC-TR; Vendorpart (none) -> USB2514B-AEZC-CT-ND
- Y1: Mfgrpart (none) -> XRCGB24M000F0L00R0; Part XRCGB24M000F0L00R0 -> (none)
